File: ESP32Template.kicad_sch (KiCad schematic)
At the start: 16 parts, among them J1 PROG, J2 JTAG, SW1 SW_Push, U1 ESP32-S3-WROOM-1-N16R8, U2 LM317_SOT-223, U3 LM317_SOT-223

Commit message: Example PCB v1
Parts:
- added D1, D2: LED, LED_THT:LED_D5.0mm, symbol Device:LED_Small
- added H1, H2: MountingHole, MountingHole:MountingHole_3.2mm_M3, symbol Mechanical:MountingHole
- added J3: Conn_01x08, FBR_Footprints:TE_776280-1, symbol Connector_Generic:Conn_01x08
- added R10, R9: 100, Resistor_THT:R_Axial_DIN0207_L6.3mm_D2.5mm_P7.62mm_Horizontal, symbol Device:R_Small
- added R6: 20k, Resistor_THT:R_Axial_DIN0207_L6.3mm_D2.5mm_P7.62mm_Horizontal, symbol Device:R
- added R7, R8: 100k, Resistor_THT:R_Axial_DIN0207_L6.3mm_D2.5mm_P7.62mm_Horizontal, symbol Device:R_Small
- added SW2, SW3: SW_Push, Button_Switch_THT:SW_PUSH_1P1T_6x3.5mm_H4.3_APEM_MJTP1243, symbol Switch:SW_Push
- added U4: MCP2551-I-P, Package_DIP:DIP-8_W7.62mm, symbol Interface_CAN_LIN:MCP2551-I-P
- C1, C2, C3, C4, C5: footprint (none) -> Capacitor_THT:C_Disc_D5.0mm_W2.5mm_P2.50mm
- J1: footprint (none) -> Connector_PinHeader_1.27mm:PinHeader_2x03_P1.27mm_Vertical
- J2: footprint (none) -> Connector_PinHeader_1.27mm:PinHeader_2x05_P1.27mm_Vertical
- R1, R2, R3, R4, R5: footprint (none) -> Resistor_THT:R_Axial_DIN0207_L6.3mm_D2.5mm_P10.16mm_Horizontal
- SW1: footprint (none) -> Button_Switch_THT:SW_PUSH_1P1T_6x3.5mm_H4.3_APEM_MJTP1243
Connections:
- net +12V: now also J3.1 (Pin_1)
- net +3V3: now also D1.2 (A), D2.2 (A), R7.1, R8.1
- net +5V: now also U4.3 (VDD)
- net GND: now also J3.4 (Pin_4), J3.5 (Pin_5), J3.6 (Pin_6), J3.7 (Pin_7), J3.8 (Pin_8), R6.2, SW2.2, SW3.2, U4.2 (VSS)
- net CAN_RX: now reaches U1.38 (IO2)
- net CAN_RX: now also U4.4 (RXD)
- net CAN_TX: now reaches U1.39 (IO1)
- net CAN_TX: now also U4.1 (TXD)
- net SW1: now reaches U1.4 (IO4)
- net SW1: now also R7.2, SW2.1
- net SW2: now reaches U1.5 (IO5)
- net SW2: now also R8.2, SW3.1
- net LED1: now reaches U1.6 (IO6)
- net LED1: now also R9.2
- net LED2: now reaches U1.7 (IO7)
- net LED2: now also R10.2
- new net: D1.1 (K), R9.1
- new net: D2.1 (K), R10.1
- new net: R6.1, U4.8 (Rs)
- new net CANH: J3.3 (Pin_3), U4.7 (CANH)
- new net CANL: J3.2 (Pin_2), U4.6 (CANL)
- no-connect marks 1 -> 2
Other:
- note added: "CAN Transceiver"
- note added: "Digital IO"
- note added: "I/O"
- note added: "Mounting"
